File: MultMixer.sch (KiCad schematic (older format))
At the start: 51 parts, among them J1 Mult IN, J10 In 3, J11 In 4, J12 In 5, J2 Conn_02x05_Odd_Even, J3 Out 1, J4 Out 2, J5 Out 4, J6 Out 3, J7 Out 5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

Commit message: relabel output
Parts:
- J13: renamed from J?; value In 2 -> Mixer Out
Changed lines of the file:
@@
 	3425 6850 3500 6850
 $Comp
-L Connector:Conn_01x02_Male J?
+L Connector:Conn_01x02_Male J13
 U 1 1 60DE3CCC
 P 10075 2925
-F 0 "J?" H 10183 3106 50  0000 C CNN
-F 1 "In 2" H 10183 3015 50  0000 C CNN
+F 0 "J13" H 10183 3106 50  0000 C CNN
+F 1 "Mixer Out" H 10183 3015 50  0000 C CNN
 F 2 "Connector_Molex:Molex_KK-254_AE-6410-02A_1x02_P2.54mm_Vertical" H 10075 2925 50  0001 C CNN
 F 3 "~" H 10075 2925 50  0001 C CNN
