File: MultMixer.kicad_pcb (KiCad board)
At the start: 2 copper layers, 67 x 150 mm, 50 parts, among them J1 Mult IN, J10 In 3, J11 In 4, J12 In 5, J2 Conn_02x05_Odd_Even, J3 Out 1, J4 Out 2, J5 Out 4, J6 Out 3, J7 Out 5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

Commit message: shuffling
Parts:
- J1, J10, J11, J12, J3, J4, J5, J6, J7, J8, J9: footprint Connector_PinHeader_2.54mm:PinHeader_1x02_P2.54mm_Vertical -> Connector_Molex:Molex_KK-254_AE-6410-02A_1x02_P2.54mm_Vertical
- moved U1 249.5 mm to (320.8, 99.1), turned to 180 degrees
- moved R6 183.4 mm to (180.5, 196.5)
- moved R5 183.1 mm to (180.4, 172.5)
- moved R2 183.0 mm to (180.0, 146.5)
- moved R3 183.0 mm to (179.9, 159.0)
- moved R4 182.8 mm to (179.9, 184.5)
- moved J3 175.4 mm to (174.5, 146.6)
- moved J4 175.4 mm to (174.5, 159.0)
- moved J5 175.4 mm to (174.5, 184.9)
- moved J6 175.4 mm to (174.9, 172.5)
- moved J7 175.4 mm to (174.9, 196.1)
- moved J12 157.7 mm to (212.0, 163.0)
- moved U2 153.8 mm to (193.0, 79.0), turned to 270 degrees
- moved J11 152.7 mm to (212.5, 143.0)
- moved J10 148.0 mm to (212.0, 123.0)
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
Commit message: update pcb
Parts:
- added J13: In 2, Connector_Molex:Molex_KK-254_AE-6410-02A_1x02_P2.54mm_Vertical, F.Cu at (235.5, 118.0)
- moved J1 193.8 mm to (174.5, 136.5)
- moved R1 164.4 mm to (189.4, 136.5)
- moved U1 126.8 mm to (195.5, 119.0), turned to 270 degrees
Changed lines of the file:
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@@
     (tracks 0)
     (zones 0)
-    (modules 50)
+    (modules 51)
     (nets 43)
   )
@@
   )
   (module Connector_Molex:Molex_KK-254_AE-6410-02A_1x02_P2.54mm_Vertical (layer F.Cu)
+    (at 235.5 118)
+    (descr "Molex KK-254 Interconnect System, old/engineering part number: AE-6410-02A example for new part number: 22-27-2021, 2 Pins (http://www.molex.com/pdm_docs/sd/022272021_sd.pdf), generated with kicad-footprint-generator")
+    (tags "connector Molex KK-254 vertical")
+    (fp_text reference J13 (at 1.27 -4.12) (layer F.SilkS)
+      (effects (font (size 1 1) (thickness 0.15)))
+    )
+    (fp_text value "In 2" (at 1.27 4.08) (layer F.Fab)
+      (effects (font (size 1 1) (thickness 0.15)))
+    )
+    (fp_text user %R (at 1.27 -2.22) (layer F.Fab)
+      (effects (font (size 1 1) (thickness 0.15)))
+    )
+    (fp_line (start -1.27 -2.92) (end -1.27 2.88) (layer F.Fab) (width 0.1))
+    (fp_line (start -1.27 2.88) (end 3.81 2.88) (layer F.Fab) (width 0.1))
+    (fp_line (start 3.81 2.88) (end 3.81 -2.92) (layer F.Fab) (width 0.1))
+    (fp_line (start 3.81 -2.92) (end -1.27 -2.92) (layer F.Fab) (width 0.1))
+    (fp_line (start -1.38 -3.03) (end -1.38 2.99) (layer F.SilkS) (width 0.12))
+    (fp_line (start -1.38 2.99) (end 3.92 2.99) (layer F.SilkS) (width 0.12))
+    (fp_line (start 3.92 2.99) (end 3.92 -3.03) (layer F.SilkS) (width 0.12))
+    (fp_line (start 3.92 -3.03) (end -1.38 -3.03) (layer F.SilkS) (width 0.12))
+    (fp_line (start -1.67 -2) (end -1.67 2) (layer F.SilkS) (width 0.12))
+    (fp_line (start -1.27 -0.5) (end -0.562893 0) (layer F.Fab) (width 0.1))
+    (fp_line (start -0.562893 0) (end -1.27 0.5) (layer F.Fab) (width 0.1))
+    (fp_line (start 0 2.99) (end 0 1.99) (layer F.SilkS) (width 0.12))
+    (fp_line (start 0 1.99) (end 2.54 1.99) (layer F.SilkS) (width 0.12))
+    (fp_line (start 2.54 1.99) (end 2.54 2.99) (layer F.SilkS) (width 0.12))
+    (fp_line (start 0 1.99) (end 0.25 1.46) (layer F.SilkS) (width 0.12))
+    (fp_line (start 0.25 1.46) (end 2.29 1.46) (layer F.SilkS) (width 0.12))
+    (fp_line (start 2.29 1.46) (end 2.54 1.99) (layer F.SilkS) (width 0.12))
+    (fp_line (start 0.25 2.99) (end 0.25 1.99) (layer F.SilkS) (width 0.12))
+    (fp_line (start 2.29 2.99) (end 2.29 1.99) (layer F.SilkS) (width 0.12))
+    (fp_line (start -0.8 -3.03) (end -0.8 -2.43) (layer F.SilkS) (width 0.12))
+    (fp_line (start -0.8 -2.43) (end 0.8 -2.43) (layer F.SilkS) (width 0.12))
+    (fp_line (start 0.8 -2.43) (end 0.8 -3.03) (layer F.SilkS) (width 0.12))
+    (fp_line (start 1.74 -3.03) (end 1.74 -2.43) (layer F.SilkS) (width 0.12))
+    (fp_line (start 1.74 -2.43) (end 3.34 -2.43) (layer F.SilkS) (width 0.12))
+    (fp_line (start 3.34 -2.43) (end 3.34 -3.03) (layer F.SilkS) (width 0.12))
+    (fp_line (start -1.77 -3.42) (end -1.77 3.38) (layer F.CrtYd) (width 0.05))
+    (fp_line (start -1.77 3.38) (end 4.31 3.38) (layer F.CrtYd) (width 0.05))
+    (fp_line (start 4.31 3.38) (end 4.31 -3.42) (layer F.CrtYd) (width 0.05))
+    (fp_line (start 4.31 -3.42) (end -1.77 -3.42) (layer F.CrtYd) (width 0.05))
+    (pad 2 thru_hole oval (at 2.54 0) (size 1.74 2.19) (drill 1.19) (layers *.Cu *.Mask)
+      (net 2 GND))
+    (pad 1 thru_hole roundrect (at 0 0) (size 1.74 2.19) (drill 1.19) (layers *.Cu *.Mask) (roundrect_rratio 0.143678)
+      (net 7 "Net-(C8-Pad1)"))
+    (model ${KISYS3DMOD}/Connector_Molex.3dshapes/Molex_KK-254_AE-6410-02A_1x02_P2.54mm_Vertical.wrl
+      (at (xyz 0 0 0))
+      (scale (xyz 1 1 1))
+      (rotate (xyz 0 0 0))
+    )
+  )
+  (module Connector_Molex:Molex_KK-254_AE-6410-02A_1x02_P2.54mm_Vertical (layer F.Cu)
     (at 212 163)
     (descr "Molex KK-254 Interconnect System, old/engineering part number: AE-6410-02A example for new part number: 22-27-2021, 2 Pins (http://www.molex.com/pdm_docs/sd/022272021_sd.pdf), generated with kicad-footprint-generator")
@@
   )
   (module Connector_Molex:Molex_KK-254_AE-6410-02A_1x02_P2.54mm_Vertical (layer F.Cu)
-    (at 20.25 19.125)
+    (at 174.46 136.5)
     (descr "Molex KK-254 Interconnect System, old/engineering part number: AE-6410-02A example for new part number: 22-27-2021, 2 Pins (http://www.molex.com/pdm_docs/sd/022272021_sd.pdf), generated with kicad-footprint-generator")
     (tags "connector Molex KK-254 vertical")
@@
   )
   (module Sonosus:DIP-14_Socket (layer F.Cu)
-    (at 320.76 99.12 180)
+    (at 195.5 119 270)
     (descr "14-lead though-hole mounted DIP package, row spacing 7.62 mm (300 mils), Socket, LongPads")
     (tags "THT DIP DIL PDIP 2.54mm 7.62mm 300mil Socket LongPads")
-    (fp_text reference U1 (at 3.81 -2.33) (layer F.SilkS)
-      (effects (font (size 1 1) (thickness 0.15)))
-    )
-    (fp_text value TL074 (at 3.81 17.57) (layer F.Fab)
+    (fp_text reference U1 (at 3.81 -2.33 90) (layer F.SilkS)
+      (effects (font (size 1 1) (thickness 0.15)))
+    )
+    (fp_text value TL074 (at 3.81 17.57 90) (layer F.Fab)
       (effects (font (size 1 1) (thickness 0.15)))
     )
@@
     (fp_line (start 9.15 16.85) (end 9.15 -1.6) (layer F.CrtYd) (width 0.05))
     (fp_line (start 9.15 -1.6) (end -1.55 -1.6) (layer F.CrtYd) (width 0.05))
-    (fp_text user %R (at 3.81 7.62) (layer F.Fab)
+    (fp_text user %R (at 3.81 7.62 90) (layer F.Fab)
       (effects (font (size 1 1) (thickness 0.15)))
     )
     (fp_arc (start 3.81 -1.33) (end 2.81 -1.33) (angle -180) (layer F.SilkS) (width 0.12))
-    (pad 14 thru_hole oval (at 7.62 0 180) (size 2.4 1.6) (drill 0.8) (layers *.Cu *.Mask)
+    (pad 14 thru_hole oval (at 7.62 0 270) (size 2.4 1.6) (drill 0.8) (layers *.Cu *.Mask)
       (net 24 "Net-(R4-Pad2)"))
-    (pad 7 thru_hole oval (at 0 15.24 180) (size 2.4 1.6) (drill 0.8) (layers *.Cu *.Mask)
+    (pad 7 thru_hole oval (at 0 15.24 270) (size 2.4 1.6) (drill 0.8) (layers *.Cu *.Mask)
       (net 23 "Net-(R3-Pad2)"))
-    (pad 13 thru_hole oval (at 7.62 2.54 180) (size 2.4 1.6) (drill 0.8) (layers *.Cu *.Mask)
+    (pad 13 thru_hole oval (at 7.62 2.54 270) (size 2.4 1.6) (drill 0.8) (layers *.Cu *.Mask)
       (net 24 "Net-(R4-Pad2)"))
-    (pad 6 thru_hole oval (at 0 12.7 180) (size 2.4 1.6) (drill 0.8) (layers *.Cu *.Mask)
+    (pad 6 thru_hole oval (at 0 12.7 270) (size 2.4 1.6) (drill 0.8) (layers *.Cu *.Mask)
       (net 23 "Net-(R3-Pad2)"))
-    (pad 12 thru_hole oval (at 7.62 5.08 180) (size 2.4 1.6) (drill 0.8) (layers *.Cu *.Mask)
+    (pad 12 thru_hole oval (at 7.62 5.08 270) (size 2.4 1.6) (drill 0.8) (layers *.Cu *.Mask)
       (net 11 "Net-(J1-Pad1)"))
-    (pad 5 thru_hole oval (at 0 10.16 180) (size 2.4 1.6) (drill 0.8) (layers *.Cu *.Mask)
+    (pad 5 thru_hole oval (at 0 10.16 270) (size 2.4 1.6) (drill 0.8) (layers *.Cu *.Mask)
       (net 11 "Net-(J1-Pad1)"))
-    (pad 11 thru_hole oval (at 7.62 7.62 180) (size 2.4 1.6) (drill 0.8) (layers *.Cu *.Mask)
+    (pad 11 thru_hole oval (at 7.62 7.62 270) (size 2.4 1.6) (drill 0.8) (layers *.Cu *.Mask)
       (net 1 -12V))
-    (pad 4 thru_hole oval (at 0 7.62 180) (size 2.4 1.6) (drill 0.8) (layers *.Cu *.Mask)
+    (pad 4 thru_hole oval (at 0 7.62 270) (size 2.4 1.6) (drill 0.8) (layers *.Cu *.Mask)
       (net 3 +12V))
-    (pad 10 thru_hole oval (at 7.62 10.16 180) (size 2.4 1.6) (drill 0.8) (layers *.Cu *.Mask)
+    (pad 10 thru_hole oval (at 7.62 10.16 270) (size 2.4 1.6) (drill 0.8) (layers *.Cu *.Mask)
       (net 11 "Net-(J1-Pad1)"))
-    (pad 3 thru_hole oval (at 0 5.08 180) (size 2.4 1.6) (drill 0.8) (layers *.Cu *.Mask)
+    (pad 3 thru_hole oval (at 0 5.08 270) (size 2.4 1.6) (drill 0.8) (layers *.Cu *.Mask)
       (net 11 "Net-(J1-Pad1)"))
-    (pad 9 thru_hole oval (at 7.62 12.7 180) (size 2.4 1.6) (drill 0.8) (layers *.Cu *.Mask)
+    (pad 9 thru_hole oval (at 7.62 12.7 270) (size 2.4 1.6) (drill 0.8) (layers *.Cu *.Mask)
       (net 25 "Net-(R5-Pad2)"))
-    (pad 2 thru_hole oval (at 0 2.54 180) (size 2.4 1.6) (drill 0.8) (layers *.Cu *.Mask)
+    (pad 2 thru_hole oval (at 0 2.54 270) (size 2.4 1.6) (drill 0.8) (layers *.Cu *.Mask)
       (net 22 "Net-(R2-Pad2)"))
-    (pad 8 thru_hole oval (at 7.62 15.24 180) (size 2.4 1.6) (drill 0.8) (layers *.Cu *.Mask)
+    (pad 8 thru_hole oval (at 7.62 15.24 270) (size 2.4 1.6) (drill 0.8) (layers *.Cu *.Mask)
       (net 25 "Net-(R5-Pad2)"))
-    (pad 1 thru_hole rect (at 0 0 180) (size 2.4 1.6) (drill 0.8) (layers *.Cu *.Mask)
+    (pad 1 thru_hole rect (at 0 0 270) (size 2.4 1.6) (drill 0.8) (layers *.Cu *.Mask)
       (net 22 "Net-(R2-Pad2)"))
     (model ${KISYS3DMOD}/Package_DIP.3dshapes/DIP-14_W7.62mm_Socket.wrl
@@
   )
   (module Sonosus:Resistor (layer F.Cu)
-    (at 31.875 89.25)
+    (at 189.38 136.5)
     (descr "Resistor, Axial_DIN0207 series, Axial, Horizontal, pin pitch=7.62mm, 0.25W = 1/4W, length*diameter=6.3*2.5mm^2, http://cdn-reichelt.de/documents/datenblatt/B400/1_4W%23YAG.pdf")
     (tags "Resistor Axial_DIN0207 series Axial Horizontal pin pitch 7.62mm 0.25W = 1/4W length 6.3mm diameter 2.5mm")

Commit message: relabel output
Parts:
- J13: value In 2 -> Mixer Out
Changed lines of the file:
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@@
       (effects (font (size 1 1) (thickness 0.15)))
     )
-    (fp_text value "In 2" (at 1.27 4.08) (layer F.Fab)
+    (fp_text value "Mixer Out" (at 1.27 4.08) (layer F.Fab)
       (effects (font (size 1 1) (thickness 0.15)))
     )

Commit message: shuffling
Parts:
- moved D3 206.5 mm to (240.6, 163.1)
- moved R7 206.5 mm to (236.1, 163.1)
- moved C6 121.1 mm to (201.0, 120.0), turned to 270 degrees
- moved C3 115.5 mm to (188.0, 91.0)
- moved C4 105.2 mm to (173.0, 75.0)
- moved C5 99.2 mm to (176.0, 125.0), turned to 90 degrees
- moved J13 61.5 mm to (212.5, 175.0)
- moved R9 5.00 mm to (197.0, 98.0)
Other:
- board size 67 x 150 mm -> 50 x 150 mm

Commit message: almost done
Parts:
- D3: footprint LED_THT:LED_D5.0mm -> Connector_Molex:Molex_KK-254_AE-6410-02A_1x02_P2.54mm_Vertical
- moved J2 206.2 mm to (210.2, 195.8)
- moved D1 187.7 mm to (207.0, 186.0)
- moved C2 185.4 mm to (200.0, 207.0)
- moved C1 183.2 mm to (200.5, 198.0)
- moved D2 182.7 mm to (207.0, 183.0)
- moved D3 78.8 mm to (174.5, 206.0)
- moved R7 70.6 mm to (180.0, 206.0)
- moved R15 0.10 mm to (189.4, 75.9)
- moved R8 0.10 mm to (197.0, 72.9)
Routing:
- net +12V: track 0.00 -> 510.1 mm
- net -12V: track 0.00 -> 177.1 mm, vias 0 -> 2
- net Net-(R2-Pad2): track 0.00 -> 147.9 mm
- net Net-(R7-Pad2): track 0.00 -> 144.2 mm
- net Net-(R6-Pad2): track 0.00 -> 143.3 mm, vias 0 -> 2
- net Net-(C7-Pad2): track 0.00 -> 134.9 mm
- net Net-(J1-Pad1): track 0.00 -> 118.9 mm, vias 0 -> 1
- net Net-(C8-Pad1): track 0.00 -> 115.5 mm
- net Net-(R4-Pad2): track 0.00 -> 62.7 mm
- net Net-(R5-Pad2): track 0.00 -> 53.0 mm, vias 0 -> 1
- net Net-(R3-Pad2): track 0.00 -> 52.8 mm, vias 0 -> 1
- net Net-(C8-Pad2): track 0.00 -> 45.4 mm, vias 0 -> 4
- net Net-(J8-Pad1): track 0.00 -> 32.6 mm
- net Net-(J9-Pad1): track 0.00 -> 32.6 mm
- net Net-(J11-Pad1): track 0.00 -> 32.6 mm, vias 0 -> 1
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- added copper zone on B.Cu, net GND
- added copper zone on F.Cu, net GND

Commit message: silksmooth
Parts:
- IN 1: renamed from J8
- IN 2: renamed from J9
- IN 3: renamed from J10
- IN 4: renamed from J11
- IN 5: renamed from J12
- MIX OUT: renamed from J13
- MULT IN: renamed from J1
- OUT 1: renamed from J3
- OUT 2: renamed from J4
- OUT 3: renamed from J6
- OUT 4: renamed from J5
- OUT 5: renamed from J7
- renumbered D3 to LED
Routing:
- net Net-(D3-Pad2): track 3.00 -> 6.72 mm
