File: MultMixer.kicad_pcb (KiCad board)
At the start: 2 copper layers, 50 x 150 mm, 51 parts, among them J2 Conn_02x05_Odd_Even, SW1 on/off, SW2 on/off, SW3 on/off, SW4 on/off, SW5 on/off, U1 TL074, U2 TL074

Commit message: silkscreen text
Other:
- board text added: "Kosmo Multiple Mixer Layout by Sonosus July 2021 Circuits from LOOK MUM NO COMPUTER CC-BY-SA 4.0"
Changed lines of the file:
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@@
   (general
     (thickness 1.6)
-    (drawings 4)
+    (drawings 5)
     (tracks 363)
     (zones 0)
@@
     )
   )
+  (gr_text "Kosmo Multiple Mixer\nLayout by Sonosus July 2021\nCircuits from LOOK MUM NO COMPUTER\nCC-BY-SA 4.0" (at 197.8 173.4 90) (layer F.SilkS)
+    (effects (font (size 1 1) (thickness 0.15)))
+  )
   (gr_line (start 167 215) (end 167 65) (layer Edge.Cuts) (width 0.05))
